Commit message: modified urdf

File: veni_vidi_vici_bot_one/description/robot_core.xacro (robot description, xacro)
@@ -6,5 +6,5 @@
     <xacro:property name="chassis_height" value="0.138"/>
     <xacro:property name="chassis_mass" value="1.0"/>
-    <xacro:property name="wheel_radius" value="0.034"/>
+    <xacro:property name="wheel_radius" value="0.051"/>
     <xacro:property name="wheel_thickness" value="0.026"/>
     <xacro:property name="wheel_mass" value="0.05"/>

Commit message: servos

File: veni_vidi_vici_bot_one/description/robot_core.xacro (robot description, xacro)
@@ -166,3 +166,47 @@
         </xacro:inertial_sphere>
     </link>
+    <!-- DOOR LINK -->
+    <joint name="door_joint" type="continuous">
+        <origin xyz="-0.20 0.13 0.13" rpy="1.57 0 0"/>
+        <parent link="base_link"/>
+        <child link="door_servo_frame"/>
+    </joint>
+    <link name="door_servo_frame">
+        <visual>
+            <geometry>
+                <cylinder radius="0.01" length="0.005"/>
+            </geometry>
+        </visual>
+        <collision>
+            <geometry>
+                <sphere radius="0.051"/>
+            </geometry>
+        </collision>
+        <inertial>
+            <mass value="0.04021467988426049"/>
+            <inertia ixx="4e-05" iyy="7e-05" izz="4e-05" ixy="-0.0" iyz="0.0" ixz="0.0"/>
+        </inertial>
+    </link>
+    <!-- RAMP LINK -->
+    <joint name="ramp_joint" type="continuous">
+        <origin xyz="-0.40 0.13 0.13" rpy="1.57 0 0"/>
+        <parent link="base_link"/>
+        <child link="ramp_servo_frame"/>
+    </joint>
+    <link name="ramp_servo_frame">
+        <visual>
+            <geometry>
+                <cylinder radius="0.01" length="0.005"/>
+            </geometry>
+        </visual>
+        <collision>
+            <geometry>
+                <sphere radius="0.051"/>
+            </geometry>
+        </collision>
+        <inertial>
+            <mass value="0.04021467988426049"/>
+            <inertia ixx="4e-05" iyy="7e-05" izz="4e-05" ixy="-0.0" iyz="0.0" ixz="0.0"/>
+        </inertial>
+    </link>
 </robot>

File: veni_vidi_vici_bot_one/description/ros2_control.xacro (robot description, xacro)
@@ -7,4 +7,6 @@
             <param name="left_wheel_name">left_wheel_joint</param>
             <param name="right_wheel_name">right_wheel_joint</param>
+            <param name="door_servo_name">door_joint</param>
+            <param name="ramp_servo_name">ramp_joint</param>
             <param name="loop_rate">30</param>
             <param name="device">/dev/ttyACM0</param>
@@ -19,6 +21,6 @@
         <joint name="left_wheel_joint">
             <command_interface name="velocity">
-                <param name="min">-10</param>
-                <param name="max">10</param>
+                <param name="min">-20</param>
+                <param name="max">20</param>
             </command_interface>
             <state_interface name="position"/>
@@ -27,6 +29,22 @@
         <joint name="right_wheel_joint">
             <command_interface name="velocity">
-                <param name="min">-10</param>
-                <param name="max">10</param>
+                <param name="min">-20</param>
+                <param name="max">20</param>
+            </command_interface>
+            <state_interface name="position"/>
+            <state_interface name="velocity"/>
+        </joint>
+        <joint name="door_joint">
+            <command_interface name="velocity">
+                <param name="min">-5</param>
+                <param name="max">5</param>
+            </command_interface>
+            <state_interface name="position"/>
+            <state_interface name="velocity"/>
+        </joint>
+        <joint name="ramp_joint">
+            <command_interface name="velocity">
+                <param name="min">-5</param>
+                <param name="max">5</param>
             </command_interface>
             <state_interface name="position"/>

Commit message: hardware interface complete

File: veni_vidi_vici_bot_one/description/robot_core.xacro (robot description, xacro)
@@ -210,3 +210,25 @@
         </inertial>
     </link>
+    <!-- COLLECTOR LINK -->
+    <joint name="collector_joint" type="continuous">
+        <origin xyz="0.20 0.13 0.13" rpy="1.57 0 0"/>
+        <parent link="base_link"/>
+        <child link="collector_servo_frame"/>
+    </joint>
+    <link name="collector_servo_frame">
+        <visual>
+            <geometry>
+                <cylinder radius="0.01" length="0.005"/>
+            </geometry>
+        </visual>
+        <collision>
+            <geometry>
+                <sphere radius="0.051"/>
+            </geometry>
+        </collision>
+        <inertial>
+            <mass value="0.04021467988426049"/>
+            <inertia ixx="4e-05" iyy="7e-05" izz="4e-05" ixy="-0.0" iyz="0.0" ixz="0.0"/>
+        </inertial>
+    </link>
 </robot>

File: veni_vidi_vici_bot_one/description/ros2_control.xacro (robot description, xacro)
@@ -9,4 +9,5 @@
             <param name="door_servo_name">door_joint</param>
             <param name="ramp_servo_name">ramp_joint</param>
+            <param name="collector_servo_name">collector_joint</param>
             <param name="loop_rate">30</param>
             <param name="device">/dev/ttyACM0</param>
@@ -51,4 +52,12 @@
             <state_interface name="velocity"/>
         </joint>
+        <joint name="collector_joint">
+            <command_interface name="velocity">
+                <param name="min">-5</param>
+                <param name="max">5</param>
+            </command_interface>
+            <state_interface name="position"/>
+            <state_interface name="velocity"/>
+        </joint>
     </ros2_control>
 </robot>
