Commit message: touched button

File: veni_vidi_vici_bot_one/description/lidar.xacro (robot description, xacro)
@@ -4,5 +4,5 @@
         <parent link="chassis"/>
         <child link="laser_frame"/>
-        <origin xyz="0.445 0 0.28" rpy="0 0 0"/>
+        <origin xyz="0.445 0.04 0.28" rpy="0 0 0"/>
     </joint>
     <link name="laser_frame">

File: veni_vidi_vici_bot_one/description/robot.urdf (robot description, URDF)
Before this commit: robot robot, 10 links, 9 joints
Links:
- added link collector_servo_frame, mass 0.04021467988426049; collision sphere radius=0.051; visual cylinder length=0.005 radius=0.01
- added link door_servo_frame, mass 0.04021467988426049; collision sphere radius=0.051; visual cylinder length=0.005 radius=0.01
- added link ramp_servo_frame, mass 0.04021467988426049; collision sphere radius=0.051; visual cylinder length=0.005 radius=0.01
Joints:
- added joint collector_joint: type continuous, parent base_link, child collector_servo_frame, origin xyz=0.20 0.13 0.13 rpy=1.57 0 0
- added joint door_joint: type continuous, parent base_link, child door_servo_frame, origin xyz=-0.20 0.13 0.13 rpy=1.57 0 0
- added joint ramp_joint: type continuous, parent base_link, child ramp_servo_frame, origin xyz=-0.40 0.13 0.13 rpy=1.57 0 0
- joint camera_joint: origin xyz=0.6 0 0.235 rpy=0 0.436332 0 -> xyz=0.615 0 0.24 rpy=0 0.436332 0
- joint laser_joint: origin xyz=0.445 0 0.28 rpy=0 0 0 -> xyz=0.445 0.04 0.28 rpy=0 0 0

File: veni_vidi_vici_bot_one/description/robot_core.xacro (robot description, xacro)
@@ -232,3 +232,25 @@
         </inertial>
     </link>
+    <!-- IMU LINK -->
+    <joint name="imu_joint" type="fixed">
+        <origin xyz="-0.16 0.05 0.20" rpy="0 0 0"/>
+        <parent link="base_link"/>
+        <child link="imu_link"/>
+    </joint>
+    <link name="imu_link">
+        <visual>
+            <geometry>
+                <cylinder radius="0.01" length="0.005"/>
+            </geometry>
+        </visual>
+        <collision>
+            <geometry>
+                <sphere radius="0.051"/>
+            </geometry>
+        </collision>
+        <inertial>
+            <mass value="0.04021467988426049"/>
+            <inertia ixx="4e-05" iyy="7e-05" izz="4e-05" ixy="-0.0" iyz="0.0" ixz="0.0"/>
+        </inertial>
+    </link>
 </robot>
