Commit message: added description

File: veni_vidi_vici_bot_one/description/camera.xacro (robot description, xacro)
@@ -4,5 +4,5 @@
         <parent link="chassis"/>
         <child link="camera_link"/>
-        <origin xyz="0.276 0 0.181" rpy="0 0 0"/>
+        <origin xyz="0.6 0 0.23" rpy="0 0 0"/>
     </joint>
     <link name="camera_link">

File: veni_vidi_vici_bot_one/description/lidar.xacro (robot description, xacro)
@@ -4,5 +4,5 @@
         <parent link="chassis"/>
         <child link="laser_frame"/>
-        <origin xyz="0.122 0 0.212" rpy="0 0 0"/>
+        <origin xyz="0.45 0 0.28" rpy="0 0 0"/>
     </joint>
     <link name="laser_frame">

File: veni_vidi_vici_bot_one/description/robot_core.xacro (robot description, xacro)
@@ -2,17 +2,18 @@
 <robot xmlns:xacro="http://www.ros.org/wiki/xacro" >
     <xacro:include filename="inertial_macros.xacro"/>
-    <xacro:property name="chassis_length" value="0.335"/>
-    <xacro:property name="chassis_width" value="0.265"/>
-    <xacro:property name="chassis_height" value="0.138"/>
-    <xacro:property name="chassis_mass" value="1.0"/>
-    <xacro:property name="wheel_radius" value="0.051"/>
-    <xacro:property name="wheel_thickness" value="0.026"/>
-    <xacro:property name="wheel_mass" value="0.05"/>
-    <xacro:property name="wheel_offset_x" value="0.226"/>
-    <xacro:property name="wheel_offset_y" value="0.166"/>
+    <xacro:property name="chassis_length" value="0.63"/>
+    <xacro:property name="chassis_width" value="0.365"/>
+    <xacro:property name="chassis_height" value="0.205"/>
+    <xacro:property name="chassis_mass" value="4.75"/>
+    <xacro:property name="wheel_radius" value="0.06"/>
+    <xacro:property name="wheel_thickness" value="0.061"/>
+    <xacro:property name="wheel_mass" value="0.160"/>
+    <xacro:property name="wheel_offset_x" value="0.43"/>
+    <xacro:property name="wheel_offset_y" value="0.22"/>
     <xacro:property name="wheel_offset_z" value="0.01"/>
-    <xacro:property name="caster_wheel_radius" value="0.01"/>
+    <xacro:property name="caster_wheel_radius" value="0.025"/>
     <xacro:property name="caster_wheel_mass" value="0.01"/>
-    <xacro:property name="caster_wheel_offset_x" value="0.075"/>
+    <xacro:property name="caster_wheel_offset_x" value="0.025"/>
+    <xacro:property name="caster_wheel_offset_y" value="0.168"/>
     <xacro:property name="caster_wheel_offset_z" value="${wheel_offset_z - wheel_radius + caster_wheel_radius}"/>
     <material name="white">
@@ -38,5 +39,5 @@
         <parent link="base_link"/>
         <child link="base_footprint"/>
-        <origin xyz="0 0 0"/>
+        <origin xyz="0 0 0" rpy="0 0 0"/>
     </joint>
     <link name="base_footprint">
@@ -66,4 +67,7 @@
         </xacro:inertial_box>
     </link>
+    <gazebo reference="chassis">
+        <material>Gazebo/Orange</material>
+    </gazebo>
     <!-- LEFT WHEEL LINK -->
     <joint name="left_wheel_joint" type="continuous">
@@ -89,4 +93,7 @@
         </xacro:inertial_cylinder>
     </link>
+    <gazebo reference="left_wheel">
+        <material>Gazebo/Blue</material>
+    </gazebo>
     <!-- RIGHT WHEEL LINK -->
     <joint name="right_wheel_joint" type="continuous">
@@ -112,11 +119,36 @@
         </xacro:inertial_cylinder>
     </link>
-    <!-- CASTER WHEEL LINK -->
-    <joint name="caster_wheel_joint" type="fixed">
+    <gazebo reference="right_wheel">
+        <material>Gazebo/Blue</material>
+    </gazebo>
+    <!--RIGHT CASTER WHEEL LINK -->
+    <joint name="right_caster_wheel_joint" type="fixed">
         <parent link="chassis"/>
-        <child link="caster_wheel"/>
-        <origin xyz="${caster_wheel_offset_x} 0 ${caster_wheel_offset_z}"/>
+        <child link="right_caster_wheel"/>
+        <origin xyz="${caster_wheel_offset_x} ${-caster_wheel_offset_y} ${caster_wheel_offset_z}"/>
     </joint>
-    <link name="caster_wheel">
+    <link name="right_caster_wheel">
+        <visual>
+            <geometry>
+                <sphere radius="${caster_wheel_radius}"/>
+            </geometry>
+            <material name="white"/>
+        </visual>
+        <collision>
+            <geometry>
+                <sphere radius="${caster_wheel_radius}"/>
+            </geometry>
+        </collision>
+        <xacro:inertial_sphere mass="${caster_wheel_mass}" radius="${caster_wheel_radius}">
+            <origin xyz="0 0 0" rpy="0 0 0"/>
+        </xacro:inertial_sphere>
+    </link>
+    <!--LEFT CASTER WHEEL LINK -->
+    <joint name="left_caster_wheel_joint" type="fixed">
+        <parent link="chassis"/>
+        <child link="left_caster_wheel"/>
+        <origin xyz="${caster_wheel_offset_x} ${caster_wheel_offset_y} ${caster_wheel_offset_z}"/>
+    </joint>
+    <link name="left_caster_wheel">
         <visual>
             <geometry>

File: veni_vidi_vici_bot_one/description/ros2_control.xacro (robot description, xacro)
@@ -8,6 +8,6 @@
             <param name="right_wheel_name">right_wheel_joint</param>
             <param name="loop_rate">30</param>
-            <param name="device">/dev/ttyACM0</param>
-            <param name="baud_rate">57600</param>
+            <param name="device">/dev/ttyUSB0</param>
+            <param name="baud_rate">9600</param>
             <param name="timeout_ms">1000</param>
             <param name="enc_counts_per_rev">3436</param>

Commit message: backup

File: veni_vidi_vici_bot_one/description/camera.xacro (robot description, xacro)
@@ -4,5 +4,5 @@
         <parent link="chassis"/>
         <child link="camera_link"/>
-        <origin xyz="0.6 0 0.23" rpy="0 0 0"/>
+        <origin xyz="0.615 0 0.24" rpy="0 0.436332 0"/>
     </joint>
     <link name="camera_link">

File: veni_vidi_vici_bot_one/description/lidar.xacro (robot description, xacro)
@@ -4,5 +4,5 @@
         <parent link="chassis"/>
         <child link="laser_frame"/>
-        <origin xyz="0.45 0 0.28" rpy="0 0 0"/>
+        <origin xyz="0.445 0 0.28" rpy="0 0 0"/>
     </joint>
     <link name="laser_frame">

File: veni_vidi_vici_bot_one/description/robot.urdf (robot description, URDF)
Before this commit: robot robot, 10 links, 9 joints
Links:
- link chassis: geometry collision box size=0.63 0.35 0.205; visual box size=0.63 0.35 0.205
Joints:
- joint camera_joint: origin xyz=0.6 0 0.23 rpy=0 0 0 -> xyz=0.6 0 0.235 rpy=0 0.436332 0
- joint laser_joint: origin xyz=0.45 0 0.28 rpy=0 0 0 -> xyz=0.445 0 0.28 rpy=0 0 0
- joint left_wheel_joint: origin xyz=0 0.22 0 rpy=-1.5707963267948966 0 0 -> xyz=0 0.2155 0 rpy=-1.5707963267948966 0 0
- joint right_wheel_joint: origin xyz=0 -0.22 0 rpy=1.5707963267948966 0 0 -> xyz=0 -0.2155 0 rpy=1.5707963267948966 0 0

File: veni_vidi_vici_bot_one/description/robot_core.xacro (robot description, xacro)
@@ -3,5 +3,5 @@
     <xacro:include filename="inertial_macros.xacro"/>
     <xacro:property name="chassis_length" value="0.63"/>
-    <xacro:property name="chassis_width" value="0.365"/>
+    <xacro:property name="chassis_width" value="0.35"/>
     <xacro:property name="chassis_height" value="0.205"/>
     <xacro:property name="chassis_mass" value="4.75"/>
@@ -10,5 +10,5 @@
     <xacro:property name="wheel_mass" value="0.160"/>
     <xacro:property name="wheel_offset_x" value="0.43"/>
-    <xacro:property name="wheel_offset_y" value="0.22"/>
+    <xacro:property name="wheel_offset_y" value="0.185"/>
     <xacro:property name="wheel_offset_z" value="0.01"/>
     <xacro:property name="caster_wheel_radius" value="0.025"/>
@@ -74,5 +74,5 @@
         <parent link="base_link"/>
         <child link="left_wheel"/>
-        <origin xyz="0 ${wheel_offset_y} 0" rpy="-${pi/2} 0 0" />
+        <origin xyz="0 ${wheel_offset_y + wheel_thickness/2} 0" rpy="-${pi/2} 0 0" />
         <axis xyz="0 0 1"/>
     </joint>
@@ -100,5 +100,5 @@
         <parent link="base_link"/>
         <child link="right_wheel"/>
-        <origin xyz="0 ${-wheel_offset_y} 0" rpy="${pi/2} 0 0" />
+        <origin xyz="0 ${-(wheel_offset_y + wheel_thickness/2)} 0" rpy="${pi/2} 0 0" />
         <axis xyz="0 0 -1"/>
     </joint>

Commit message: saved description

File: veni_vidi_vici_bot_one/description/camera.xacro (robot description, xacro)
@@ -4,5 +4,5 @@
         <parent link="chassis"/>
         <child link="camera_link"/>
-        <origin xyz="0.615 0 0.24" rpy="0 0.436332 0"/>
+        <origin xyz="0.615 0.0 0.24" rpy="0 0.35 0"/>
     </joint>
     <link name="camera_link">

File: veni_vidi_vici_bot_one/description/lidar.xacro (robot description, xacro)
@@ -4,5 +4,5 @@
         <parent link="chassis"/>
         <child link="laser_frame"/>
-        <origin xyz="0.445 0.04 0.28" rpy="0 0 0"/>
+        <origin xyz="0.445 0.01 0.28" rpy="0 0 0"/>
     </joint>
     <link name="laser_frame">
